File: v2/charging.brd (EAGLE design)
At the start: 53.8 x 48.5 mm, 37 parts, among them Q1 CSD16301Q2, Q2 CSD16301Q2, U1 MCP73871-2CCI/ML, U2 MCP1824ST-3302E/DB, U3 TPS61090, U4 BQ29718

Commit message: update
Parts:
- Q1, Q2: value CSD16301Q2 -> (none)
Changed lines of the file:
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@@
 <layer number="25" name="tNames" color="7" fill="1" visible="yes" active="yes"/>
 <layer number="26" name="bNames" color="7" fill="1" visible="yes" active="yes"/>
-<layer number="27" name="tValues" color="7" fill="1" visible="yes" active="yes"/>
+<layer number="27" name="tValues" color="7" fill="1" visible="no" active="yes"/>
 <layer number="28" name="bValues" color="7" fill="1" visible="yes" active="yes"/>
 <layer number="29" name="tStop" color="7" fill="3" visible="no" active="yes"/>
@@
 <text x="3.048" y="40.132" size="1.778" layer="25">+</text>
 <text x="2.54" y="33.528" size="1.778" layer="25">-</text>
-<text x="9.652" y="10.922" size="1.27" layer="25" rot="R180">PROG2</text>
+<text x="6.35" y="13.208" size="1.27" layer="25" rot="R180">PROG2</text>
 <text x="0.508" y="13.97" size="1.27" layer="25">SEL</text>
 <text x="0.762" y="16.256" size="1.27" layer="25">TE</text>
@@
 <text x="42.672" y="45.974" size="1.27" layer="25">-</text>
 <text x="38.862" y="46.228" size="1.27" layer="25">LO</text>
-<text x="29.718" y="47.498" size="1.778" layer="25" rot="R180">G FIERRO 7/19/2016
+<text x="17.526" y="47.244" size="1.016" layer="25" rot="R180">G FIERRO 7/19/2016
 CHARGER v2</text>
 </plain>
@@
 <attribute name="PACKAGE" value="QFN-20" x="19.304" y="16.51" size="1.778" layer="27" display="off"/>
 </element>
-<element name="U2" library="Microchip_By_element14_Batch_1" package="SOT230P700X180-4N" value="MCP1824ST-3302E/DB" x="6.35" y="27.686" rot="R180">
+<element name="U2" library="Microchip_By_element14_Batch_1" package="SOT230P700X180-4N" value="MCP1824ST-3302E/DB" x="6.35" y="27.686" smashed="yes" rot="R180">
 <attribute name="MPN" value="MCP1824ST-3302E/DB" x="6.35" y="27.686" size="1.778" layer="27" rot="R180" display="off"/>
 <attribute name="OC_FARNELL" value="1578379" x="6.35" y="27.686" size="1.778" layer="27" rot="R180" display="off"/>
@@
 <attribute name="OC_NEWARK" value="05N1293" x="6.35" y="27.686" size="1.778" layer="27" rot="R180" display="off"/>
 <attribute name="PACKAGE" value="SOT-223-3" x="6.35" y="27.686" size="1.778" layer="27" rot="R180" display="off"/>
+<attribute name="NAME" x="4.5974" y="21.844" size="2.0828" layer="25" ratio="10" rot="SR0"/>
+<attribute name="VALUE" x="12.065" y="33.5534" size="2.0828" layer="27" ratio="10" rot="SR180"/>
 </element>
 <element name="R11" library="resistor" package="R0603" value="0 ohm" x="9.398" y="19.05" smashed="yes" rot="R180">
@@
 </element>
 <element name="R13" library="resistor" package="R0603" value="0" x="9.398" y="12.954" smashed="yes" rot="R180">
-<attribute name="NAME" x="7.747" y="12.319" size="1.27" layer="25" rot="R180"/>
+<attribute name="NAME" x="7.493" y="11.811" size="1.27" layer="25" rot="R180"/>
 <attribute name="VALUE" x="10.033" y="14.859" size="1.27" layer="27" rot="R180"/>
 </element>
@@
 </element>
 <element name="U4" library="insole" package="6-WFDFN" value="BQ29718" x="34.798" y="17.272"/>
-<element name="Q1" library="insole" package="6-SMD" value="CSD16301Q2" x="30.48" y="8.636" smashed="yes" rot="R90">
+<element name="Q1" library="insole" package="6-SMD" value="" x="30.48" y="8.636" smashed="yes" rot="R90">
 <attribute name="NAME" x="31.75" y="7.366" size="1.27" layer="25" rot="R180"/>
 <attribute name="VALUE" x="34.29" y="7.366" size="1.27" layer="25" rot="R90"/>
 </element>
-<element name="Q2" library="insole" package="6-SMD" value="CSD16301Q2" x="35.306" y="8.636" smashed="yes" rot="R90">
+<element name="Q2" library="insole" package="6-SMD" value="" x="35.306" y="8.636" smashed="yes" rot="R90">
 <attribute name="NAME" x="36.576" y="7.112" size="1.27" layer="25" rot="R180"/>
 <attribute name="VALUE" x="39.116" y="7.366" size="1.27" layer="25" rot="R90"/>
