File: v2/charging.sch (EAGLE design)
At the start: 37 parts, among them Q1 CSD16301Q2, Q2 CSD16301Q2, U1 MCP73871-2CCI/ML, U2 MCP1824ST-3302E/DB, U3 TPS61090, U4 BQ29718

Commit message: update
Changed lines of the file:
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@@
 <part name="R14" library="resistor" deviceset="R-US_" device="R0603" value="0"/>
 <part name="U4" library="insole" deviceset="BQ29718" device=""/>
-<part name="Q1" library="insole" deviceset="CSD16301Q2" device=""/>
-<part name="Q2" library="insole" deviceset="CSD16301Q2" device=""/>
+<part name="Q1" library="insole" deviceset="CSD16301Q2" device="" value=""/>
+<part name="Q2" library="insole" deviceset="CSD16301Q2" device="" value=""/>
 <part name="R15" library="resistor" deviceset="R-US_" device="R0805" value="330"/>
 <part name="C8" library="resistor" deviceset="C-EU" device="C0805" value="0.1uF"/>
